File: schematics/z80 RPM/z80 RPM.kicad_pcb (KiCad board)
At the start: 2 copper layers, 88.9 x 57.1 mm, 37 parts, among them J1 Conn_01x08, J10 Conn_01x04, J11 Conn_01x02, J12 Conn_01x08, J13 Conn_02x02_Counter_Clockwise, J14 Conn_02x02_Counter_Clockwise, J2 Conn_01x08, J3 Conn_01x16, J4 Conn_01x04, J5 Conn_01x02, J6 Conn_01x08, J7 Conn_01x08, J8 Conn_01x16, J9 Conn_01x08, SW1 SW_SPST, U1 z80 CPU, U2 27C512, U4 74LS138, U5 74LS32, U6 24M512, X1 GTXO-14T

Commit message: design updated to v1.1
Parts:
- added R3: 2k, Resistor_THT:R_Axial_DIN0207_L6.3mm_D2.5mm_P10.16mm_Horizontal, F.Cu at (62.2, 29.5)
- added R4: 2k, Resistor_THT:R_Axial_DIN0207_L6.3mm_D2.5mm_P10.16mm_Horizontal, F.Cu at (49.9, 29.5)
- moved H2 10.0 mm to (60.7, 33.7)
- moved H3 10.0 mm to (60.7, 78.7)
- renumbered C7 to C2, C6 to C3, C2 to C4, C3 to C5, C4 to C6, C5 to C7, H3 to H1, H1 to H3, J11 to J10, J2 to J11, J7 to J2, J6 to J3, J9 to J4, J3 to J5, J8 to J6, J4 to J7, J10 to J8, J5 to J9, U2 to U1, U6 to U2, U1 to U3, U5 to U4, U4 to U5
Routing:
- net Net-(JP1-B): track 13.4 -> 54.8 mm, vias 0 -> 1
- net Net-(JP2-B): track 12.6 -> 43.2 mm, vias 0 -> 1
- net /A15: track 84.8 -> 82.9 mm
- net /A14: track 88.6 -> 87.1 mm
- net /D0: track 121.4 -> 120.2 mm
- net /~{RESET}: track 134.0 -> 133.4 mm
Other:
- board size 88.9 x 57.1 mm -> 89 x 57 mm
- board text added: "Oct 2024"
- board text added: "z80 Rapid Prototyping Module v1.1"
- board text removed: "27C512"
- board text removed: "Jun 2024"
- board text removed: "z80 Rapid Prototyping Module"
