File: schematics/z80 RPM/z80 RPM.kicad_sch (KiCad schematic)
At the start: 37 parts, among them J1 Conn_01x08, J10 Conn_01x04, J11 Conn_01x02, J12 Conn_01x08, J13 Conn_02x02_Counter_Clockwise, J14 Conn_02x02_Counter_Clockwise, J2 Conn_01x08, J3 Conn_01x16, J4 Conn_01x04, J5 Conn_01x02, J6 Conn_01x08, J7 Conn_01x08, J8 Conn_01x16, J9 Conn_01x08, SW1 SW_SPST, U1 z80 CPU, U2 27C512, U4 74LS138, U5 74LS32, U6 24M512, X1 GTXO-14T

Commit message: design updated to v1.1
Parts:
- added R3, R4: 2k, Resistor_THT:R_Axial_DIN0207_L6.3mm_D2.5mm_P10.16mm_Horizontal, symbol Device:R
- renumbered C7 to C2, C6 to C3, C2 to C4, C3 to C5, C4 to C6, C5 to C7, H3 to H1, H1 to H3, J11 to J10, J2 to J11, J7 to J2, J6 to J3, J9 to J4, J3 to J5, J8 to J6, J4 to J7, J10 to J8, J5 to J9, U2 to U1, U6 to U2, U1 to U3, U5 to U4, U4 to U5
Connections:
- net GND: now also R3.2, R4.2
- net at JP2.2 (B), U4.4: now also R3.1
- net at JP1.2 (B), U4.1: now also R4.1
Other:
- title: z80 RPM v1.0 -> z80 RPM v1.1
- moved on the sheet: JP1, JP2, U4A, U4B
